Commit message: stefano

File: robotiq_85_description/urdf/robotiq_85_gripper.urdf.xacro (robot description, xacro)
@@ -34,5 +34,5 @@
             <kd>1.0</kd>
         </gazebo>
-        <joint name="${prefix}gripper_finger1_joint" type="revolute">
+        <joint name="${prefix}gripper_finger1_joint" type="fixed">
             <parent link="${prefix}gripper_base_link"/>
             <child link="${prefix}gripper_finger1_knuckle_link"/>
@@ -41,5 +41,5 @@
             <limit lower="0.0" upper="0.804" velocity="2.0" effort="1000"/>
         </joint>
-        <joint name="${prefix}gripper_finger2_joint" type="revolute">
+        <joint name="${prefix}gripper_finger2_joint" type="fixed">
             <parent link="${prefix}gripper_base_link"/>
             <child link="${prefix}gripper_finger2_knuckle_link"/>
@@ -47,5 +47,5 @@
             <origin rpy="0.0 0.0 0.0" xyz="0.05490451627 -0.03060114443 0.0"/>
             <limit lower="-3.14" upper="3.14" velocity="100.0" effort="1000"/>
-            <mimic joint="${prefix}gripper_finger1_joint"/>
+<!--             <mimic joint="${prefix}gripper_finger1_joint"/> -->
         </joint>
         <link name="${prefix}gripper_finger1_knuckle_link">
@@ -163,5 +163,5 @@
             <kd>1.0</kd>
         </gazebo>
-        <joint name="${prefix}gripper_finger1_inner_knuckle_joint" type="continuous">
+        <joint name="${prefix}gripper_finger1_inner_knuckle_joint" type="fixed">
             <parent link="${prefix}gripper_base_link"/>
             <child link="${prefix}gripper_finger1_inner_knuckle_link"/>
@@ -169,7 +169,7 @@
             <origin xyz="0.06142 0.0127 0" rpy="${pi} 0.0 0.0" />
             <limit lower="-3.14" upper="3.14" velocity="100.0" effort="0.1"/>
-            <mimic joint="${prefix}gripper_finger1_joint" offset="0"/>
-        </joint>
-        <joint name="${prefix}gripper_finger2_inner_knuckle_joint" type="continuous">
+<!--             <mimic joint="${prefix}gripper_finger1_joint" offset="0"/> -->
+        </joint>
+        <joint name="${prefix}gripper_finger2_inner_knuckle_joint" type="fixed">
             <parent link="${prefix}gripper_base_link"/>
             <child link="${prefix}gripper_finger2_inner_knuckle_link"/>
@@ -177,5 +177,5 @@
             <origin xyz="0.06142 -0.0127 0" rpy="0 0 0"/>
             <limit lower="-3.14" upper="3.14" velocity="100.0" effort="0.1"/>
-            <mimic joint="${prefix}gripper_finger1_joint" offset="0"/>
+<!--             <mimic joint="${prefix}gripper_finger1_joint" offset="0"/> -->
         </joint>
         <link name="${prefix}gripper_finger1_inner_knuckle_link">
@@ -231,5 +231,5 @@
             <kd>1.0</kd>
         </gazebo>
-        <joint name="${prefix}gripper_finger1_finger_tip_joint" type="continuous">
+        <joint name="${prefix}gripper_finger1_finger_tip_joint" type="fixed">
             <parent link="${prefix}gripper_finger1_inner_knuckle_link"/>
             <child link="${prefix}gripper_finger1_finger_tip_link"/>
@@ -237,7 +237,7 @@
             <origin xyz="0.04303959807 -0.03759940821 0.0" rpy="0.0 0.0 0.0"/>
             <limit lower="-3.14" upper="3.14" velocity="100.0" effort="0.1"/>
-            <mimic joint="${prefix}gripper_finger1_joint" multiplier="-1"/>
-        </joint>
-        <joint name="${prefix}gripper_finger2_finger_tip_joint" type="continuous">
+<!--             <mimic joint="${prefix}gripper_finger1_joint" multiplier="-1"/> -->
+        </joint>
+        <joint name="${prefix}gripper_finger2_finger_tip_joint" type="fixed">
             <parent link="${prefix}gripper_finger2_inner_knuckle_link"/>
             <child link="${prefix}gripper_finger2_finger_tip_link"/>
@@ -245,5 +245,5 @@
             <origin rpy="0.0 0.0 0.0" xyz="0.04303959807 -0.03759940821  0.0"/>
             <limit lower="-3.14" upper="3.14" velocity="100.0" effort="0.1"/>
-            <mimic joint="${prefix}gripper_finger1_joint" multiplier="-1"/>
+<!--             <mimic joint="${prefix}gripper_finger1_joint" multiplier="-1"/> -->
         </joint>
         <link name="${prefix}gripper_finger1_finger_tip_link">
